File: pcb/ai_hat_adda.sch (EAGLE design)
At the start: 285 parts, among them J1 1X01-SM, J10 1X01-SM, J100 1X01-SM, J101 1X01-SM, J102 1X01-SM, J103 1X01-SM, J104 1X01-SM, J105 1X01-SM, J106 1X01-SM, J107 1X01-SM, J108 1X01-SM, J109 1X01-SM, J11 1X01-SM, J110 1X01-SM, J111 1X01-SM, J112 1X01-SM, J113 1X01-SM, J114 1X01-SM, J115 1X01-SM, J116 1X01-SM, J117 1X01-SM, J118 1X01-SM, J119 1X01-SM, J12 1X01-SM, J120 1X01-SM, J121 1X01-SM, J122 1X01-SM, J123 1X01-SM, J124 1X01-SM, J125 1X01-SM, J126 1X01-SM, J127 1X01-SM, J128 1X01-SM, J129 1X01-SM, J13 1X01-SM, J130 1X01-SM, J131 1X01-SM, J132 1X01-SM, J133 1X01-SM, J134 1X01-SM, J135 1X01-SM, J136 1X01-SM, J137 1X01-SM, J138 1X01-SM, J139 1X01-SM, J14 1X01-SM, J140 1X01-SM, J141 1X01-SM, J142 1X01-SM, J143 1X01-SM, J144 1X01-SM, J145 1X01-SM, J146 1X01-SM, J147 1X01-SM, J148 1X01-SM, J149 1X01-SM, J15 1X01-SM, J150 1X01-SM, J151 1X01-SM, J152 1X01-SM, J153 1X01-SM, J154 1X01-SM, J155 1X01-SM, J156 1X01-SM, J157 1X01-SM, J158 1X01-SM, J159 1X01-SM, J16 1X01-SM, J160 1X01-SM, J161 1X01-SM, J162 1X01-SM, J163 1X01-SM, J164 1X01-SM, J165 1X01-SM, J166 1X01-SM, J167 1X01-SM, J168 1X01-SM, J169 1X01-SM, J17 1X01-SM, J170 1X01-SM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

Commit message: latest update
Parts:
- removed J10, J100, J101, J102, J103, J104, J105, J106, J107, J108, J109, J11, J110, J111, J112, J113, J114, J115, J116, J117, J118, J119, J12, J120, J121, J122, J123, J124, J125, J126, J127, J128, J129, J13, J130, J131, J132, J133, J134, J135, J136, J137, J138, J139, J14, J140, J141, J142, J143, J144, J145, J146, J147, J148, J149, J15, J150, J151, J152, J153, J154, J155, J156, J157, J158, J159, J16, J160, J161, J162, J163, J164, J165, J166, J167, J168, J169, J17, J170, J171, J172, J173, J174, J175, J176, J177, J178, J179, J180, J181, J182, J183, J184, J185, J186, J187, J188, J189, J190, J191, J192, J193, J194, J195, J196, J197, J198, J199, J20, J200, J201, J202, J203, J204, J205, J206, J207, J208, J209, J21, J210, J211, J212, J213, J214, J215, J216, J217, J218, J219, J22, J220, J221, J222, J223, J224, J225, J226, J227, J228, J229, J23, J230, J231, J232, J233, J234, J235, J236, J237, J238, J239, J24, J240, J241, J242, J243, J244, J245, J246, J247, J248, J249, J25, J250, J26, J27, J28, J29, J30, J31, J32, J33, J34, J35, J36, J37, J38, J39, J40, J41, J42, J43, J44, J45, J46, J47, J48, J49, J5, J50, J51, J52, J53, J54, J55, J56, J57, J58, J59, J6, J60, J61, J62, J63, J64, J65, J66, J67, J68, J69, J7, J70, J71, J72, J73, J74, J75, J76, J77, J78, J79, J8, J80, J81, J82, J83, J84, J85, J86, J87, J88, J89, J9, J90, J91, J92, J93, J94, J95, J96, J97, J98, J99: 1X01-SM, Ai_Connectors:1X01-SM
- removed J18: JST-3P-MALE, Ai_Connectors:JST-3P-MALE
- removed J19: JST-4P-MALE, Ai_Connectors:JST-4P-MALE
- added C2, C3, C4: 0.1uF, Ai_Passives:CAP0402
- added C5: 10uF, Ai_Passives:CAP0402
- added R5, R6: 10K, Ai_Passives:RES0402
- added U2: ADS1115, Ai_IC:ADS1115
- added U3, U4: MCP4725, SparkFun-AnalogIC:MCP4725SOT-23
- J1, J2: value 1X01-SM -> 1X03ST; device Ai_Connectors:1X01-SM -> Ai_Connectors:1X03ST
- J3, J4: value 1X01-SM -> 1X02ST; device Ai_Connectors:1X01-SM -> Ai_Connectors:1X02ST
- R4: value 300 -> 10K; device Ai_Passives:RES0603 -> Ai_Passives:RES0402
Connections:
- removed net 2: J18.2, R4.2
- removed net N$10: J55.1, J56.1, J57.1, J58.1, J59.1
- removed net N$11: J62.1, J63.1, J64.1, J65.1, J66.1
- removed net N$12: J69.1, J70.1, J71.1, J72.1, J73.1
- removed net N$13: J76.1, J77.1, J78.1, J79.1, J80.1
- removed net N$14: J83.1, J84.1, J85.1, J86.1, J87.1
- removed net N$15: J90.1, J91.1, J92.1, J93.1, J94.1
- removed net N$16: J100.1, J101.1, J97.1, J98.1, J99.1
- removed net N$17: J104.1, J105.1, J106.1, J107.1, J108.1
- removed net N$18: J111.1, J112.1, J113.1, J114.1, J115.1
- removed net N$19: J120.1, J121.1, J122.1, J123.1, J124.1
- removed net N$20: J127.1, J128.1, J129.1, J130.1, J131.1
- removed net N$21: J134.1, J135.1, J136.1, J137.1, J138.1
- removed net N$22: J141.1, J142.1, J143.1, J144.1, J145.1
- removed net N$23: J148.1, J149.1, J150.1, J151.1, J152.1
- removed net N$24: J155.1, J156.1, J157.1, J158.1, J159.1
- removed net N$25: J162.1, J163.1, J164.1, J165.1, J166.1
- removed net N$26: J169.1, J170.1, J171.1, J172.1, J173.1
- removed net N$27: J176.1, J177.1, J178.1, J179.1, J180.1
- removed net N$28: J183.1, J184.1, J185.1, J186.1, J187.1
- removed net N$29: J190.1, J191.1, J192.1, J193.1, J194.1
- removed net N$30: J197.1, J198.1, J199.1, J200.1, J201.1
- removed net N$31: J204.1, J205.1, J206.1, J207.1, J208.1
- removed net N$32: J211.1, J212.1, J213.1, J214.1, J215.1
- removed net N$33: J218.1, J219.1, J220.1, J221.1, J222.1
- removed net N$34: J225.1, J226.1, J227.1, J228.1, J229.1
- removed net N$35: J232.1, J233.1, J234.1, J235.1, J236.1
- removed net N$36: J239.1, J240.1, J241.1, J242.1, J243.1
- removed net N$37: J246.1, J247.1, J248.1, J249.1, J250.1
- removed net N$5: J20.1, J21.1, J22.1, J23.1, J24.1
- removed net N$6: J27.1, J28.1, J29.1, J30.1, J31.1
- removed net N$7: J34.1, J35.1, J36.1, J37.1, J38.1
- removed net N$8: J41.1, J42.1, J43.1, J44.1, J45.1
- removed net N$9: J48.1, J49.1, J50.1, J51.1, J52.1
- new net AIN0: J1.1, U2.AIN0
- new net AIN1: J1.2, U2.AIN1
- new net AIN2: J1.3, U2.AIN2
- new net AIN3: J2.1, U2.AIN3
- new net ALERT: U2.ALERT/RDY
- new net AOUT0: J2.2, U3.VOUT
- new net AOUT1: J2.3, U4.VOUT
- net #18: no longer R4.1
- net 3V3: now also C2.1, C3.1, C4.1, C5.2, U2.VDD, U3.VDD, U4.VDD; no longer J102.1, J109.1, J116.1, J118.1, J125.1, J132.1, J139.1, J146.1, J153.1, J160.1, J167.1, J174.1, J181.1, J188.1, J195.1, J202.1, J209.1, J216.1, J223.1, J230.1, J237.1, J244.1
- net 5V: now also J3.2; no longer J16.1, J18.1, J19.1, J25.1, J32.1, J39.1, J46.1, J53.1, J60.1, J67.1, J74.1, J81.1, J88.1, J95.1
- net GND: now also C2.2, C3.2, C4.2, C5.1, J3.1, R4.1, R5.1, R6.1, U2.VSS, U3.VSS, U4.VSS; no longer J103.1, J110.1, J117.1, J119.1, J126.1, J133.1, J140.1, J147.1, J154.1, J161.1, J168.1, J17.1, J175.1, J18.3, J182.1, J189.1, J19.4, J196.1, J203.1, J210.1, J217.1, J224.1, J231.1, J238.1, J245.1, J26.1, J33.1, J40.1, J47.1, J54.1, J61.1, J68.1, J75.1, J82.1, J89.1, J96.1
- net MOSI: no longer J19.3
- net N$1: now also R4.2, U2.ADDR; no longer J1.1, J2.1, J3.1, J4.1, J5.1
- net N$2: now also R6.2, U4.AO; no longer J10.1, J6.1, J7.1, J8.1, J9.1
- net N$4: now also R5.2, U3.AO; no longer J11.1, J12.1, J13.1, J14.1, J15.1
- net SCK: no longer J19.2
- net SCL: now also J4.1, U2.SCL, U3.SCL, U4.SCL
- net SDA: now also J4.2, U2.SDA, U3.SDA, U4.SDA
Other:
- moved on the sheet: C1, CFG, K1, R1, R2, R3, R4, U1
